Commit message: 改造(2026-10-17): 美化圆柱机器人 + 加装IMU/相机/6路超声波 + 多层建筑世界(支撑柱/静止汽车/二层) + 随包三层地图 + 航点巡航 + Nav2参数调优 + 三项目导航选型分析
- URDF: 全局材质调色板/饰环/信标/相机云台/超声波阵列, 碰撞与惯性保持原验证参数
- 传感器: gz插件+桥接+ultrasonic_node(Range+点云, 角速度门控), gz_frame_id源头修frame
- 世界: building_world.sdf(24x16m两层) + room_world.sdf随包安装, world参数化launch
- 地图: building_floor1(SLAM实测)/building_floor2(CAD导出)/room 随包
- 验证: room世界Nav2 3/3目标SUCCEEDED; 建筑一层SLAM 8/8航点; 巡航23/23航点
- 文档: 导航算法选型分析/改造说明/实机接入指南§12(传感器实机接入契约)

File: src/datarobot_description/urdf/databot/actuator/wheel.urdf.xacro (robot description, xacro)
@@ -2,18 +2,21 @@
 <robot xmlns:xacro="http://www.ros.org/wiki/xacro" >
     <xacro:macro name="wheel_xacro" params="wheel_name xyz radius:=0.083">
-        <!-- 机器人的轮子 -->
+        <!-- 机器人的轮子：橡胶胎 + 银色轮毂 双层外观 -->
         <link name="${wheel_name}_link">
-            <!-- 部件的外观描述 -->
-            <visual>
-                <!-- 沿着自己几何中心的偏移和旋转量 -->
+            <!-- 外观：外胎 -->
+            <visual name="tire">
                 <origin xyz="0.0 0.0 0.0" rpy="1.57079 0.0 0.0"/>
-                <!-- 几何形状 -->
                 <geometry>
                     <cylinder radius="${radius}" length="0.06"/>
                 </geometry>
-                <!-- 颜色材质 -->
-                <material name="wheel_blue">
-                    <color rgba="1.0 0.0 1.0 0.8"/>
-                </material>
+                <material name="mat_tire"/>
+            </visual>
+            <!-- 外观：轮毂（比外胎略宽，从两侧都能看到银色盘面）-->
+            <visual name="hub">
+                <origin xyz="0.0 0.0 0.0" rpy="1.57079 0.0 0.0"/>
+                <geometry>
+                    <cylinder radius="${radius * 0.6}" length="0.064"/>
+                </geometry>
+                <material name="mat_silver"/>
             </visual>
             <!-- 碰撞体描述（用于 Gazebo 物理仿真）-->

File: src/datarobot_description/urdf/databot/base.urdf.xacro (robot description, xacro)
@@ -1,4 +1,36 @@
 <?xml version="1.0"?>
 <robot xmlns:xacro="http://www.ros.org/wiki/xacro" >
+    <!-- 全局材质调色板：所有子文件只按名字引用，颜色改这一处即可。
+         注意 alpha 全部为 1.0：半透明车体会让 Gazebo 里的渲染出现透视串面 -->
+    <material name="mat_body">
+        <color rgba="0.92 0.93 0.95 1.0"/>   <!-- 珠白车身 -->
+    </material>
+    <material name="mat_accent">
+        <color rgba="0.10 0.35 0.65 1.0"/>   <!-- 科技蓝饰环 -->
+    </material>
+    <material name="mat_dark">
+        <color rgba="0.16 0.17 0.20 1.0"/>   <!-- 深灰：裙边/顶盖/传感器舱 -->
+    </material>
+    <material name="mat_orange">
+        <color rgba="0.95 0.45 0.05 1.0"/>   <!-- 警示橙：顶部信标 -->
+    </material>
+    <material name="mat_panel">
+        <color rgba="0.08 0.08 0.09 1.0"/>   <!-- 前脸面板 -->
+    </material>
+    <material name="mat_silver">
+        <color rgba="0.75 0.76 0.78 1.0"/>   <!-- 轮毂/镜头圈 -->
+    </material>
+    <material name="mat_tire">
+        <color rgba="0.13 0.13 0.14 1.0"/>   <!-- 橡胶轮胎 -->
+    </material>
+    <material name="mat_lidar">
+        <color rgba="0.22 0.23 0.25 1.0"/>   <!-- 激光雷达 -->
+    </material>
+    <material name="mat_imu">
+        <color rgba="0.00 0.40 0.20 1.0"/>   <!-- IMU 模块 PCB 绿 -->
+    </material>
+    <material name="mat_us">
+        <color rgba="0.10 0.15 0.45 1.0"/>   <!-- 超声波模块 深蓝 -->
+    </material>
     <!-- base_height: base_link 高出地面的高度, 由 datarobot.urdf.xacro 统一算出并传入
          (= -wheel_z + wheel_radius). 地平面只在那一处决定, 从动轮等部件的 z
@@ -16,20 +48,70 @@
         <!-- 机器人的身体部分 -->
         <link name="base_link">
-            <!-- 部件的外观描述 -->
-            <visual>
-                <!-- 沿着自己几何中心的偏移和旋转量 -->
+            <!-- ===== 外观（美化版：白塔身 + 蓝饰环 + 深灰顶盖 + 橙色信标）===== -->
+            <!-- 主塔身：圆柱轮廓保持不变，碰撞/惯性在下方单独定义 -->
+            <visual name="body">
                 <origin xyz="0.0 0.0 0.716" rpy="0.0 0.0 0.0"/>
-                <!-- 几何形状 -->
                 <geometry>
-                    <!-- 圆柱体半径 高度 -->
                     <cylinder radius="${radius}" length="${length}"/>
                 </geometry>
-                <!-- 颜色材质 -->
-                <material name="white">
-                    <color rgba="1.0 1.0 1.0 0.5"/>
-                </material>
+                <material name="mat_body"/>
+            </visual>
+            <!-- 底部裙边：盖住轮舱接缝 -->
+            <visual name="skirt">
+                <origin xyz="0.0 0.0 0.02" rpy="0.0 0.0 0.0"/>
+                <geometry>
+                    <cylinder radius="${radius + 0.005}" length="0.12"/>
+                </geometry>
+                <material name="mat_dark"/>
+            </visual>
+            <!-- 上下两道蓝色饰环 -->
+            <visual name="ring_lower">
+                <origin xyz="0.0 0.0 0.55" rpy="0.0 0.0 0.0"/>
+                <geometry>
+                    <cylinder radius="${radius + 0.006}" length="0.05"/>
+                </geometry>
+                <material name="mat_accent"/>
+            </visual>
+            <visual name="ring_upper">
+                <origin xyz="0.0 0.0 1.30" rpy="0.0 0.0 0.0"/>
+                <geometry>
+                    <cylinder radius="${radius + 0.006}" length="0.05"/>
+                </geometry>
+                <material name="mat_accent"/>
+            </visual>
+            <!-- 前脸面板：标识车头方向 -->
+            <visual name="front_panel">
+                <origin xyz="${radius - 0.002} 0.0 0.95" rpy="0.0 0.0 0.0"/>
+                <geometry>
+                    <box size="0.024 0.30 0.45"/>
+                </geometry>
+                <material name="mat_panel"/>
+            </visual>
+            <!-- 顶盖 -->
+            <visual name="top_cap">
+                <origin xyz="0.0 0.0 ${length - 0.109}" rpy="0.0 0.0 0.0"/>
+                <geometry>
+                    <cylinder radius="${radius + 0.005}" length="0.05"/>
+                </geometry>
+                <material name="mat_dark"/>
+            </visual>
+            <!-- 顶部信标底座 + 灯 -->
+            <visual name="beacon_base">
+                <origin xyz="0.0 0.0 ${length - 0.0715}" rpy="0.0 0.0 0.0"/>
+                <geometry>
+                    <cylinder radius="0.09" length="0.025"/>
+                </geometry>
+                <material name="mat_dark"/>
+            </visual>
+            <visual name="beacon">
+                <origin xyz="0.0 0.0 ${length - 0.024}" rpy="0.0 0.0 0.0"/>
+                <geometry>
+                    <cylinder radius="0.045" length="0.07"/>
+                </geometry>
+                <material name="mat_orange"/>
             </visual>
             <!-- 碰撞体描述（用于 Gazebo 物理仿真）-->
-            <!-- 使用更矮的碰撞体来降低重心,避免倒地 -->
+            <!-- 使用更矮的碰撞体来降低重心,避免倒地.
+                 ⚠️ 碰撞几何是历史验证过的（重心/倾覆/雷达遮挡特性都依赖它），美化不动它 -->
             <collision>
                 <origin xyz="0.0 0.0 0.25" rpy="0.0 0.0 0.0"/>

File: src/datarobot_description/urdf/databot/datarobot.urdf.xacro (robot description, xacro)
@@ -1,5 +1,5 @@
 <?xml version="1.0"?>
 <robot xmlns:xacro="http://www.ros.org/wiki/xacro" name="databot">
-<!-- 基础部分 -->
+<!-- 基础部分（含全局材质调色板） -->
 <xacro:include filename="$(find datarobot_description)/urdf/databot/base.urdf.xacro"/>
 <!-- 传感器部分 -->
@@ -7,4 +7,5 @@
 <xacro:include filename="$(find datarobot_description)/urdf/databot/senser/camera.urdf.xacro"/>
 <xacro:include filename="$(find datarobot_description)/urdf/databot/senser/laser.urdf.xacro"/>
+<xacro:include filename="$(find datarobot_description)/urdf/databot/senser/ultrasonic.urdf.xacro"/>
 <!-- 执行器部分 -->
 <xacro:include filename="$(find datarobot_description)/urdf/databot/actuator/wheel.urdf.xacro"/>
@@ -23,7 +24,19 @@
 <xacro:property name="caster_radius" value="0.083"/>
 <xacro:base_xacro length="1.70" radius="0.28" base_height="${base_height}"/>
+<!-- IMU：装在车体中轴顶部内腔（实机对应主控板上方的 IMU 模块） -->
 <xacro:imu_xacro xyz="0.0 0.0 0.02"/>
-<xacro:camera_xacro xyz="0.0 0.0 1.566"/>
+<!-- 顶部云台相机：顶盖前沿，下俯 10°。camera_enabled:=false 可关掉传感器渲染省算力 -->
+<xacro:arg name="camera_enabled" default="true"/>
+<xacro:camera_xacro xyz="0.20 0.0 1.656" rpy="0.0 -0.17 0.0" enabled="$(arg camera_enabled)"/>
+<!-- 激光雷达：车头外伸支架上，x=0.30 在车体半径(0.28)之外，避免自遮挡 -->
 <xacro:laser_xacro xyz="0.30 0.0 0.0"/>
+<!-- 超声波 ×6：z=-0.13 → 离地约 0.12 m，专管激光盲区以下的低矮障碍
+     （车位挡轮杆、路缘等）。前 3 + 左右各 1 + 后 1，覆盖全向 -->
+<xacro:ultrasonic_xacro name="us_front"        xyz="0.283 0.0 -0.13"    yaw="0.0"/>
+<xacro:ultrasonic_xacro name="us_front_left"   xyz="0.20 0.20 -0.13"    yaw="0.7854"/>
+<xacro:ultrasonic_xacro name="us_front_right"  xyz="0.20 -0.20 -0.13"   yaw="-0.7854"/>
+<xacro:ultrasonic_xacro name="us_left"         xyz="0.0 0.283 -0.13"    yaw="1.5708"/>
+<xacro:ultrasonic_xacro name="us_right"        xyz="0.0 -0.283 -0.13"   yaw="-1.5708"/>
+<xacro:ultrasonic_xacro name="us_rear"         xyz="-0.283 0.0 -0.13"   yaw="3.14159"/>
 <xacro:wheel_xacro wheel_name="left_wheel"
                    xyz="0 0.179 ${wheel_z}" radius="${wheel_radius}"/>

File: src/datarobot_description/urdf/databot/gazebo.urdf.xacro (robot description, xacro)
@@ -45,8 +45,6 @@
             <maxVel>1.0</maxVel>
         </gazebo>
-        <!-- 为 base_link 设置材质颜色 -->
-        <gazebo reference="base_link">
-            <material>Gazebo/White</material>
-        </gazebo>
+        <!-- 车体材质不再用 <gazebo reference> 覆盖：
+             URDF 里的材质已改为不透明成品色，sdformat 转换会直接带进 gz 渲染 -->
     </xacro:macro>
     <!-- 关节状态发布插件 -->

File: src/datarobot_description/urdf/databot/senser/camera.urdf.xacro (robot description, xacro)
@@ -1,27 +1,55 @@
 <?xml version="1.0"?>
 <robot xmlns:xacro="http://www.ros.org/wiki/xacro" >
-    <xacro:macro name="camera_xacro" params="xyz">
-        <!-- 顶端摄像头 -->
+    <xacro:macro name="camera_xacro" params="xyz rpy:='0 0 0' enabled:=true">
+        <!-- 顶端摄像头（云台造型：深灰舱体 + 银色镜头圈）-->
         <link name="camera_link">
-            <!-- 部件的外观描述 -->
-            <visual>
-                <!-- 沿着自己几何中心的偏移和旋转量 -->
+            <visual name="pod">
                 <origin xyz="0.0 0.0 0.0" rpy="0.0 0.0 0.0"/>
-                <!-- 几何形状 -->
                 <geometry>
-                    <box size="0.1 0.1 0.1"/>
+                    <box size="0.10 0.10 0.08"/>
                 </geometry>
-                <!-- 颜色材质 -->
-                <material name="camera_white">
-                    <color rgba="0.0 0.0 0.0 0.5"/>
-                </material>
+                <material name="mat_dark"/>
+            </visual>
+            <visual name="lens">
+                <origin xyz="0.055 0.0 0.0" rpy="0.0 1.57079 0.0"/>
+                <geometry>
+                    <cylinder radius="0.025" length="0.02"/>
+                </geometry>
+                <material name="mat_silver"/>
             </visual>
         </link>
-        <!-- 机器人的关节，用于组合机器人的部件 -->
+        <!-- 机器人的关节，用于组合机器人的部件。
+             rpy 支持俯仰（如 0 -0.17 0 = 下俯 10°），默认水平朝前 -->
         <joint name="camera_joint" type="fixed">
             <parent link="base_link"/>
             <child link="camera_link"/>
-            <origin xyz="${xyz}" rpy="0.0 0.0 0.0"/>
+            <origin xyz="${xyz}" rpy="${rpy}"/>
         </joint>
+        <!-- Gazebo 相机传感器：桥接后出 /camera/image_raw + /camera/camera_info。
+             不加 <topic>，用与雷达一致的 gz 默认作用域话题（启动文件按 world 名拼路径）。
+             enabled:=false 时不挂传感器（CPU 紧张的导航测试省一路渲染负载） -->
+        <xacro:if value="${enabled}">
+            <gazebo reference="camera_link">
+                <sensor name="camera_sensor" type="camera">
+                    <pose>0 0 0 0 0 0</pose>
+                    <always_on>1</always_on>
+                    <update_rate>5</update_rate>
+                    <visualize>false</visualize>
+                    <gz_frame_id>camera_link</gz_frame_id>
+                    <camera>
+                        <horizontal_fov>1.2</horizontal_fov>
+                        <image>
+                            <width>320</width>
+                            <height>240</height>
+                            <format>R8G8B8</format>
+                        </image>
+                        <clip>
+                            <near>0.05</near>
+                            <far>30</far>
+                        </clip>
+                    </camera>
+                </sensor>
+            </gazebo>
+        </xacro:if>
     </xacro:macro>
 </robot>

File: src/datarobot_description/urdf/databot/senser/imu.urdf.xacro (robot description, xacro)
@@ -2,19 +2,22 @@
 <robot xmlns:xacro="http://www.ros.org/wiki/xacro" >
     <xacro:macro name="imu_xacro" params="xyz">
-        <!-- 机器人的imu部分 惯性测量传感器 -->
+        <!-- 机器人的IMU部分 惯性测量传感器 -->
         <link name="imu_link">
-            <!-- 部件的外观描述 -->
+            <!-- 外观：PCB 小模块 -->
             <visual>
-                <!-- 沿着自己几何中心的偏移和旋转量 -->
                 <origin xyz="0.0 0.0 0.0" rpy="0.0 0.0 0.0"/>
-                <!-- 几何形状 -->
                 <geometry>
                     <box size="0.02 0.02 0.02"/>
                 </geometry>
-                <!-- 颜色材质 -->
-                <material name="white">
-                    <color rgba="1.0 1.0 0.0 0.5"/>
-                </material>
+                <material name="mat_imu"/>
             </visual>
+            <!-- 惯性参数：传感器本体很轻，球体近似 -->
+            <inertial>
+                <origin xyz="0.0 0.0 0.0" rpy="0.0 0.0 0.0"/>
+                <mass value="0.02"/>
+                <inertia ixx="1e-06" ixy="0.0" ixz="0.0"
+                         iyy="1e-06" iyz="0.0"
+                         izz="1e-06"/>
+            </inertial>
         </link>
         <!-- 机器人的关节，用于组合机器人的部件 -->
@@ -24,4 +27,15 @@
             <origin xyz="${xyz}" rpy="0.0 0.0 0.0"/>
         </joint>
+        <!-- Gazebo IMU 传感器插件（gz-sim-imu-system 需在 world 里加载）.
+             不加 <topic>：桥接用 gz-sim 默认作用域话题 .../imu_sensor/imu，两边名字一致不会断流。
+             <gz_frame_id> 让消息直接带 imu_link 坐标系，省掉 ROS 侧改 frame 的补丁节点 -->
+        <gazebo reference="imu_link">
+            <sensor name="imu_sensor" type="imu">
+                <always_on>1</always_on>
+                <update_rate>50</update_rate>
+                <visualize>false</visualize>
+                <gz_frame_id>imu_link</gz_frame_id>
+            </sensor>
+        </gazebo>
     </xacro:macro>
 </robot>

File: src/datarobot_description/urdf/databot/senser/laser.urdf.xacro (robot description, xacro)
@@ -2,18 +2,21 @@
 <robot xmlns:xacro="http://www.ros.org/wiki/xacro" >
     <xacro:macro name="laser_xacro" params="xyz">
-        <!-- 激光雷达 -->
+        <!-- 激光雷达：深灰筒身 + 支架 -->
         <link name="laser_link">
-            <!-- 部件的外观描述 -->
+            <!-- 外观：雷达本体 -->
             <visual>
-                <!-- 沿着自己几何中心的偏移和旋转量 -->
                 <origin xyz="0.0 0.0 -0.01" rpy="0.0 0.0 0.0"/>
-                <!-- 几何形状 -->
                 <geometry>
                     <cylinder radius="0.0275" length="0.055"/>
                 </geometry>
-                <!-- 颜色材质 -->
-                <material name="white">
-                    <color rgba="1.0 1.0 0.0 0.5"/>
-                </material>
+                <material name="mat_lidar"/>
+            </visual>
+            <!-- 外观：从车身表面伸出的支架 -->
+            <visual name="bracket">
+                <origin xyz="-0.045 0.0 -0.01" rpy="0.0 0.0 0.0"/>
+                <geometry>
+                    <box size="0.07 0.04 0.04"/>
+                </geometry>
+                <material name="mat_dark"/>
             </visual>
             <!-- 碰撞体描述（用于 Gazebo 物理仿真）-->
@@ -43,6 +46,8 @@
         </joint>
         <!-- Gazebo 激光雷达传感器.
-             不要加 <topic> 覆盖话题名: 启动文件里的桥接用的是 gz-sim 默认的
-             作用域名 .../laser_sensor/scan, 一旦指定 topic 桥接就订阅不到 -->
+             不要加 <topic> 覆盖话题名: 桥接用的是 gz-sim 默认的作用域名
+             .../laser_sensor/scan, 一旦指定 topic 桥接就订阅不到.
+             <gz_frame_id> 让 ROS 侧 LaserScan 直接带 laser_link 坐标系，
+             不再需要 frame 修正补丁节点 -->
         <gazebo reference="laser_link">
             <sensor name="laser_sensor" type="gpu_lidar">
@@ -50,4 +55,5 @@
                 <visualize>true</visualize>
                 <update_rate>10</update_rate>
+                <gz_frame_id>laser_link</gz_frame_id>
                 <lidar>
                     <scan>
